File: KiCad/MM32.kicad_pcb (KiCad board)
At the start: 4 copper layers, 22 x 22 mm, 18 parts, among them J1 MICROMOD-2222, U1 MK20DX256VLH7, U2 MKL02Z32VFG4, Y1 16MHz, Y2 16MHz

Commit message: cleanup
Parts:
- added e: LOGO, Project:logo, B.Cu at (141.2, 57.5)
Other:
- board text added: "lunOptics MM32 V2.1 (2020-12)"
- board text removed: "lunOptics MicroMod_32 2020-12 V2.0"
