File: KiCad/MM32.sch (KiCad schematic (older format))
At the start: 18 parts, among them J1 MICROMOD-2222, U1 MK20DX256VLH7, U2 MKL02Z32VFG4, Y1 16MHz, Y2 16MHz

Commit message: Rename KiCad files
Changed lines of the file:
@@
 L power:GND #PWR04
 U 1 1 5F944AFD
-P 2675 5450
-F 0 "#PWR04" H 2675 5200 50  0001 C CNN
-F 1 "GND" V 2680 5322 50  0000 R CNN
-F 2 "" H 2675 5450 50  0001 C CNN
-F 3 "" H 2675 5450 50  0001 C CNN
-	1    2675 5450
+P 2650 5450
+F 0 "#PWR04" H 2650 5200 50  0001 C CNN
+F 1 "GND" V 2655 5322 50  0000 R CNN
+F 2 "" H 2650 5450 50  0001 C CNN
+F 3 "" H 2650 5450 50  0001 C CNN
+	1    2650 5450
 	0    1    1    0
 $EndComp
@@
 	0    1    1    0
 $EndComp
+Wire Wire Line
+	2650 5450 2675 5450
 $EndSCHEMATC

Commit message: cleanup
Parts:
- U1: symbol TeensyMM-rescue:MK20DX256VLH7-TeensyDIY -> TeensyDIY:MK20DX256VLH7
- U2: symbol TeensyMM-rescue:TeensyBootloader_MKL02Z32VFG4-TeensyDIY -> TeensyDIY:TeensyBootloader_MKL02Z32VFG4
Changed lines of the file:
@@
 	9425 1700 9425 1750
 $Comp
-L TeensyMM-rescue:MK20DX256VLH7-TeensyDIY U1
+L TeensyDIY:MK20DX256VLH7 U1
 U 1 1 5FD41634
 P 8175 3650
@@
 $EndComp
 $Comp
-L TeensyMM-rescue:TeensyBootloader_MKL02Z32VFG4-TeensyDIY U2
+L TeensyDIY:TeensyBootloader_MKL02Z32VFG4 U2
 U 1 1 5FD47E0F
 P 13075 4600
